Commit message: refine structure

File: hardwares/urdf/ur.urdf.xacro (robot description, xacro)
@@ -49,5 +49,5 @@
     safety_k_position="$(arg safety_k_position)"
     >
-     <origin xyz="0 0 0" rpy="0 0 0" />          <!-- position robot in the world -->
+     <origin xyz="0 0 0" rpy="0 0 3.14159265358979323846" />          <!-- position robot in the world -->
   </xacro:ur_robot>
 </robot>
